Commit message: update v1.1.4 :update neo_gazebo package (using unified entrance) :update neo_moveit_package (supported multi devices) :moveit + gazebo basically completion

File: neo_description/urdf/EndEffector/AG95/dh_robotics_ag95.gazebo.xacro (robot description, xacro)
@@ -50,5 +50,5 @@
       <joint>gripper_finger1_joint</joint>
       <mimicJoint>gripper_finger1_finger_tip_joint</mimicJoint>
-      <multiplier>1.49462955</multiplier>
+      <multiplier>0.49462955</multiplier>
       <offset>0.0</offset>
     </plugin>

File: neo_description/urdf/EndEffector/AG95/dh_robotics_ag95.urdf.xacro (robot description, xacro)
@@ -11,5 +11,5 @@
   <xacro:macro name="ag95_gripper" params="connected_to *origin">
 <!-- /////////////////////////////////////////////  flange   //////////////////////////////////////////////////// -->
-    <joint name="${connected_to}_to_gripper_base_link" type="fixed">
+    <joint name="connected_joint" type="fixed">
       <xacro:insert_block name="origin" />
       <parent link="${connected_to}" />
@@ -101,5 +101,5 @@
       <origin rpy="0.0 0.0 0.0" xyz="0.016  0 0.10586 "/>
       <limit lower="-3.14" upper="3.14" velocity="100.0" effort="1000"/>
-      <mimic joint="gripper_finger1_joint"/>
+      <mimic joint="gripper_finger1_joint"  multiplier="1"/>
     </joint>
     <link name="gripper_finger2_knuckle_link">
@@ -131,5 +131,5 @@
       <origin xyz="0.0292080077784 0.0 -0.0227132622407" rpy="0 0 0" />
       <limit lower="-3.14" upper="3.14" velocity="100.0" effort="0.1"/>
-      <mimic joint="gripper_finger1_joint" />
+      <mimic joint="gripper_finger1_joint" multiplier="0.4563942"/>
     </joint>
     <link name="gripper_finger1_finger_link">
@@ -161,5 +161,5 @@
         <origin xyz="0.0292080077784 0.0 -0.0227132622407" rpy="0 0 0" />
         <limit lower="-3.14" upper="3.14" velocity="100.0" effort="0.1"/>
-        <mimic joint="gripper_finger1_joint" />
+        <mimic joint="gripper_finger1_joint" multiplier="0.4563942"/>
     </joint>
     <link name="gripper_finger2_finger_link">
@@ -191,5 +191,5 @@
       <origin rpy="0.0 0.0 3.14" xyz="-0.016 0 0.10586"/>
       <limit lower="-3.14" upper="3.14" velocity="100.0" effort="0.1"/>
-      <mimic joint="gripper_finger1_joint" />
+      <mimic joint="gripper_finger1_joint" multiplier="1.49462955"/>
     </joint>
     <link name="gripper_finger1_inner_knuckle_link">
@@ -221,5 +221,5 @@
         <origin rpy="0.0 0.0 0.0" xyz="0.016 0 0.10586"/>
         <limit lower="-3.14" upper="3.14" velocity="100.0" effort="0.1"/>
-        <mimic joint="gripper_finger1_joint" />
+        <mimic joint="gripper_finger1_joint" multiplier="1.49462955"/>
       </joint>
     <link name="gripper_finger2_inner_knuckle_link">
@@ -251,5 +251,5 @@
       <origin xyz="0.0394969463769 0.0 0.0382752038125 " rpy="0.0 0.0 0.0"/>
       <limit lower="-3.14" upper="3.14" velocity="100.0" effort="0.1"/>
-      <mimic joint="gripper_finger1_joint" />
+      <mimic joint="gripper_finger1_joint" multiplier="1.49462955"/>
     </joint>
     <link name="gripper_finger1_finger_tip_link">
@@ -281,5 +281,5 @@
       <origin xyz="0.0394969463769 0.0 0.0382752038125 " rpy="0.0 0.0 0.0"/>
       <limit lower="-3.14" upper="3.14" velocity="100.0" effort="0.1"/>
-      <mimic joint="gripper_finger1_joint" />
+      <mimic joint="gripper_finger1_joint" multiplier="1.49462955"/>
     </joint>
     <link name="gripper_finger2_finger_tip_link">

File: neo_description/urdf/NX63A1/NX63A1_with_ag95.urdf.xacro (robot description, xacro)
@@ -1,4 +1,4 @@
 <?xml version="1.0"?>
-<robot xmlns:xacro="http://ros.org/wiki/xacro" name="NX63A1" >
+<robot xmlns:xacro="http://ros.org/wiki/xacro" name="NX63A1_with_ag95" >
   <!-- common stuff -->
   <xacro:include filename="$(find neo_description)/urdf/common.gazebo.xacro" />
@@ -7,6 +7,4 @@
   <!-- AG95 -->
   <xacro:include filename="$(find neo_description)/urdf/EndEffector/AG95/dh_robotics_ag95.urdf.xacro" />
-  <!-- D435 -->
-  <xacro:include filename="$(find neo_description)/urdf/Sensor/D435/realsense_d435.urdf.xacro" />
   <!-- world link -->
   <link name="world" />
@@ -19,7 +17,3 @@
   	<origin xyz="-0.042 -0.042 0" rpy="0 0 0" />
   </xacro:ag95_gripper>
-  <!-- sensor -->
-  <xacro:realsense_d435 connected_to="ag95_flange_link">
-    <origin xyz="0.087 0.042 0" rpy="0 0 3.1415"/>
-  </xacro:realsense_d435>
 </robot>

File: neo_description/urdf/NX63A1/NX63A1_with_ag95_d435.urdf.xacro (robot description, xacro)
@@ -1,4 +1,4 @@
 <?xml version="1.0"?>
-<robot xmlns:xacro="http://ros.org/wiki/xacro" name="NX63A1" >
+<robot xmlns:xacro="http://ros.org/wiki/xacro" name="NX63A1_with_ag95_d435" >
   <!-- common stuff -->
   <xacro:include filename="$(find neo_description)/urdf/common.gazebo.xacro" />
@@ -7,4 +7,6 @@
   <!-- AG95 -->
   <xacro:include filename="$(find neo_description)/urdf/EndEffector/AG95/dh_robotics_ag95.urdf.xacro" />
+  <!-- D435 -->
+  <xacro:include filename="$(find neo_description)/urdf/Sensor/D435/realsense_d435.urdf.xacro" />
   <!-- world link -->
   <link name="world" />
@@ -17,3 +19,7 @@
   	<origin xyz="-0.042 -0.042 0" rpy="0 0 0" />
   </xacro:ag95_gripper>
+  <!-- sensor -->
+  <xacro:realsense_d435 connected_to="ag95_flange_link">
+    <origin xyz="0.087 0.042 0" rpy="0 0 3.1415"/>
+  </xacro:realsense_d435>
 </robot>

File: neo_moveit_config/config/NX63A1/NX63A1.xacro (robot description, xacro)
@@ -1,8 +1,5 @@
-<?xml version="1.0" ?>
-<!--This does not replace URDF, and is not an extension of URDF.
-    This is a format for representing semantic information about the robot structure.
-    A URDF file must exist for this robot as well, where the joints and the links that are referenced are defined
--->
-<robot name="NX63A1">
+<?xml version='1.0' encoding='utf-8'?>
+<robot xmlns:xacro="http://www.ros.org/wiki/xacro" name="NX63A1">
+  <xacro:macro name="NX63A1">
     <!--GROUPS: Representation of a set of joints and links. This can be useful for specifying DOF to plan for, defining arms, end effectors, etc-->
     <!--LINKS: When a link is specified, the parent joint of that link (if it exists) is automatically included-->
@@ -10,27 +7,27 @@
     <!--CHAINS: When a chain is specified, all the links along the chain (including endpoints) are included in the group. Additionally, all the joints that are parents to included links are also included. This means that joints along the chain and the parent joint of the base link are included in the group-->
     <!--SUBGROUPS: Groups can also be formed by referencing to already defined group names-->
-    <group name="manipulator">
-        <chain base_link="base_link" tip_link="ee_flange_link" />
+    <group name="NX63A1">
+      <chain base_link="base_link" tip_link="ee_link" />
     </group>
     <!--GROUP STATES: Purpose: Define a named state for a particular group, in terms of joint values. This is useful to define states like 'folded arms'-->
-    <group_state name="home" group="manipulator">
-        <joint name="fifth_joint" value="0" />
-        <joint name="first_joint" value="0" />
-        <joint name="fourth_joint" value="0" />
-        <joint name="second_joint" value="0" />
-        <joint name="sixth_joint" value="0" />
-        <joint name="third_joint" value="0" />
+    <group_state name="home" group="NX63A1">
+      <joint name="fifth_joint" value="0" />
+      <joint name="first_joint" value="0" />
+      <joint name="fourth_joint" value="0" />
+      <joint name="second_joint" value="0" />
+      <joint name="sixth_joint" value="0" />
+      <joint name="third_joint" value="0" />
     </group_state>
     <!--END EFFECTOR: Purpose: Represent information about an end effector.-->
     <!-- end_effector name="moveit_ee" parent_link="ee_flange_link" group="endeffector" / -->
     <!--DISABLE COLLISIONS: By default it is assumed that any link of the robot could potentially come into collision with any other link in the robot. This tag disables collision checking between a specified pair of links. -->
-    <disable_collisions link1="base_link" link2="ee_flange_link" reason="Never" />
+    <disable_collisions link1="base_link" link2="ee_link" reason="Never" />
     <disable_collisions link1="base_link" link2="first_link" reason="Adjacent" />
     <disable_collisions link1="base_link" link2="second_link" reason="Never" />
-    <disable_collisions link1="ee_flange_link" link2="fifth_link" reason="Never" />
-    <disable_collisions link1="ee_flange_link" link2="first_link" reason="Never" />
-    <disable_collisions link1="ee_flange_link" link2="fourth_link" reason="Never" />
-    <disable_collisions link1="ee_flange_link" link2="sixth_link" reason="Adjacent" />
-    <disable_collisions link1="ee_flange_link" link2="third_link" reason="Never" />
+    <disable_collisions link1="ee_link" link2="fifth_link" reason="Never" />
+    <disable_collisions link1="ee_link" link2="first_link" reason="Never" />
+    <disable_collisions link1="ee_link" link2="fourth_link" reason="Never" />
+    <disable_collisions link1="ee_link" link2="sixth_link" reason="Adjacent" />
+    <disable_collisions link1="ee_link" link2="third_link" reason="Never" />
     <disable_collisions link1="fifth_link" link2="fourth_link" reason="Adjacent" />
     <disable_collisions link1="fifth_link" link2="sixth_link" reason="Adjacent" />
@@ -41,3 +38,4 @@
     <disable_collisions link1="second_link" link2="third_link" reason="Adjacent" />
     <disable_collisions link1="sixth_link" link2="third_link" reason="Never" />
+  </xacro:macro>
 </robot>
